Commit message: 更新URDF文件以使用现代ROS命名空间和xacro属性
- 将所有URDF文件中的XML命名空间从playerstage.sourceforge.net更新为www.ros.org
- 将旧的<property>标签替换为<xacro:property>以符合现代xacro语法
- 修复r2c_legs.display.urdf.xacro中错误的include路径语法
- 将xacro宏调用方式从自闭合标签改为显式宏定义
- 为所有xacro文件生成对应的URDF XML文件
- 保持机器人名称和功能不变，仅更新语法和命名空间

File: r2_description/robots/r2.display.urdf.xacro (robot description, xacro)
@@ -1,8 +1,9 @@
 <?xml version="1.0" ?>
-<robot name="r2" xmlns:controller="http://playerstage.sourceforge.net/gazebo/xmlschema/#controller"
-			xmlns:interface="http://playerstage.sourceforge.net/gazebo/xmlschema/#interface"
-			xmlns:sensor="http://playerstage.sourceforge.net/gazebo/xmlschema/#sensor"
-			xmlns:xacro="http://playerstage.sourceforge.net/gazebo/xmlschema/#interface">
-  <property name="robot_name" value= "/r2/" />
+<robot name="r2" xmlns:controller="http://www.ros.org/wiki/controller"
+			xmlns:interface="http://www.ros.org/wiki/interface"
+			xmlns:sensor="http://www.ros.org/wiki/sensor"
+			xmlns:xacro="http://www.ros.org/wiki/xacro">
+  <!-- <property name="robot_name" value= "/r2/" /> -->
+  <xacro:property name="robot_name" value= "/r2/"/>
   <include filename="$(find r2_description)/robots/r2.urdf.xacro" />
   <include filename="$(find r2_description)/urdf/r2.gazebo.xacro" />

File: r2_description/robots/r2.sim.urdf.xacro (robot description, xacro)
@@ -1,8 +1,9 @@
 <?xml version="1.0" ?>
-<robot name="r2" xmlns:controller="http://playerstage.sourceforge.net/gazebo/xmlschema/#controller"
-			xmlns:interface="http://playerstage.sourceforge.net/gazebo/xmlschema/#interface"
-			xmlns:sensor="http://playerstage.sourceforge.net/gazebo/xmlschema/#sensor"
-			xmlns:xacro="http://playerstage.sourceforge.net/gazebo/xmlschema/#interface">
-  <property name="robot_name" value= "/r2/" />
+<robot name="r2" xmlns:controller="http://www.ros.org/wiki/controller"
+			xmlns:interface="http://www.ros.org/wiki/interface"
+			xmlns:sensor="http://www.ros.org/wiki/sensor"
+			xmlns:xacro="http://www.ros.org/wiki/xacro">
+  <!-- <property name="robot_name" value= "/r2/" /> -->
+  <xacro:property name="robot_name" value= "/r2/"/>
   <include filename="$(find r2_description)/robots/r2.urdf.xacro" />
   <include filename="$(find r2_description)/urdf/r2.gazebo.xacro" />

File: r2_description/robots/r2.urdf.xacro (robot description, xacro)
@@ -1,5 +1,6 @@
 <?xml version="1.0" ?>
-<robot name="r2">
-  <property name="robot_name" value= "/r2/" />
+<robot name="r2" xmlns:xacro="http://www.ros.org/wiki/xacro">
+  <!-- <property name="robot_name" value= "/r2/" /> -->
+  <xacro:property name="robot_name" value= "/r2/"/>
   <include filename="$(find r2_description)/urdf/models/r2.common.xacro" />
   <include filename="$(find r2_description)/urdf/models/r2.base.xacro" />

File: r2_description/robots/r2_orocos.sim.urdf.xacro (robot description, xacro)
@@ -1,8 +1,9 @@
 <?xml version="1.0" ?>
-<robot name="r2_orocos" xmlns:controller="http://playerstage.sourceforge.net/gazebo/xmlschema/#controller"
-			xmlns:interface="http://playerstage.sourceforge.net/gazebo/xmlschema/#interface"
-			xmlns:sensor="http://playerstage.sourceforge.net/gazebo/xmlschema/#sensor"
-			xmlns:xacro="http://playerstage.sourceforge.net/gazebo/xmlschema/#interface">
-  <property name="robot_name" value= "/r2/" />
+<robot name="r2_orocos" xmlns:controller="http://www.ros.org/wiki/controller"
+			xmlns:interface="http://www.ros.org/wiki/interface"
+			xmlns:sensor="http://www.ros.org/wiki/sensor"
+      xmlns:xacro="http://www.ros.org/wiki/xacro">
+  <!-- <property name="robot_name" value= "/r2/" /> -->
+  <xacro:property name="robot_name" value= "/r2/"/>
   <include filename="$(find r2_description)/urdf/models/r2c_upper_body.urdf.xacro" />
   <include filename="$(find r2_description)/urdf/r2.gazebo.xacro" />

File: r2_description/robots/r2c_full_body.sim.urdf.xacro (robot description, xacro)
@@ -1,10 +1,12 @@
 <?xml version="1.0" ?>
-<robot name="r2c_full_body" xmlns:controller="http://playerstage.sourceforge.net/gazebo/xmlschema/#controller"
-			xmlns:interface="http://playerstage.sourceforge.net/gazebo/xmlschema/#interface"
-			xmlns:sensor="http://playerstage.sourceforge.net/gazebo/xmlschema/#sensor"
-			xmlns:xacro="http://playerstage.sourceforge.net/gazebo/xmlschema/#interface">
-  <property name="robot_name" value= "/r2/" />
+<robot name="r2c_full_body" xmlns:controller="http://www.ros.org/wiki/controller"
+			xmlns:interface="http://www.ros.org/wiki/interface"
+			xmlns:sensor="http://www.ros.org/wiki/sensor"
+			xmlns:xacro="http://www.ros.org/wiki/xacro">
+  <!-- <property name="robot_name" value= "/r2/" /> -->
+  <xacro:property name="robot_name" value= "/r2/"/>
   <link name="world"/>
-  <property name="robot_name" value= "/r2/" />
+  <!-- <property name="robot_name" value= "/r2/" /> -->
+  <xacro:property name="robot_name" value= "/r2/"/>
   <!--  transforms in first joint don't seem to work properly-->
   <joint name="${robot_name}fixed/world/world_ref" type="fixed">
@@ -14,7 +16,9 @@
   </joint>
   <include filename="$(find r2_description)/urdf/models/r2c_full_body_no_world.urdf.xacro" />
-  <xacro:robot_world_origin>
+  <!-- <xacro:robot_world_origin> -->
+  <xacro:macro name="robot_world_origin">
     <origin rpy="0 0 0" xyz="0.0 0.0 1.5"/>
-  </xacro:robot_world_origin>
+  </xacro:macro>
+  <!-- </xacro:robot_world_origin> -->
   <include filename="$(find r2_description)/urdf/r2.gazebo.xacro" />
   <include filename="$(find r2_description)/urdf/sensors/r2.gazebo.sensors.xacro" />

File: r2_description/robots/r2c_full_body.urdf.xacro (robot description, xacro)
@@ -1,10 +1,11 @@
 <?xml version="1.0" ?>
-  <robot xmlns:sensor="http://playerstage.sourceforge.net/gazebo/xmlschema/#sensor"
-       xmlns:controller="http://playerstage.sourceforge.net/gazebo/xmlschema/#controller"
-       xmlns:interface="http://playerstage.sourceforge.net/gazebo/xmlschema/#interface"
-       xmlns:xacro="http://playerstage.sourceforge.net/gazebo/xmlschema/#interface"
+  <robot xmlns:sensor="http://www.ros.org/wiki/sensor"
+       xmlns:controller="http://www.ros.org/wiki/controller"
+       xmlns:interface="http://www.ros.org/wiki/interface"
+       xmlns:xacro="http://www.ros.org/wiki/xacro"
        name="r2c_full_body" >
   <link name="world"/>
-  <property name="robot_name" value= "/r2/" />
+  <!-- <property name="robot_name" value= "/r2/" /> -->
+  <xacro:property name="robot_name" value= "/r2/"/>
 <!--  transforms in first joint don't seem to work properly-->
   <joint name="${robot_name}fixed/world/robot_world" type="fixed">
@@ -14,6 +15,8 @@
   </joint>
   <include filename="$(find r2_description)/robots/r2c_full_body_no_world.urdf.xacro" />
-  <xacro:robot_base_origin>
+  <!-- <xacro:robot_base_origin> -->
+   <xacro:macro name="robot_base_origin">
     <origin xyz="0 0 1.4" rpy="0 0 0" />
-  </xacro:robot_base_origin>
+  <!-- </xacro:robot_base_origin> -->
+  </xacro:macro>
 </robot>

File: r2_description/robots/r2c_full_body_ISS.sim.urdf.xacro (robot description, xacro)
@@ -1,13 +1,16 @@
 <?xml version="1.0" ?>
-<robot name="r2c_full_body" xmlns:controller="http://playerstage.sourceforge.net/gazebo/xmlschema/#controller"
-			xmlns:interface="http://playerstage.sourceforge.net/gazebo/xmlschema/#interface"
-			xmlns:sensor="http://playerstage.sourceforge.net/gazebo/xmlschema/#sensor"
-			xmlns:xacro="http://playerstage.sourceforge.net/gazebo/xmlschema/#interface">
-  <property name="robot_name" value= "/r2/" />
+<robot name="r2c_full_body" xmlns:controller="http://www.ros.org/wiki/controller"
+			xmlns:interface="http://www.ros.org/wiki/interface"
+			xmlns:sensor="http://www.ros.org/wiki/sensor"
+			xmlns:xacro="http://www.ros.org/wiki/xacro">
+  <!-- <property name="robot_name" value= "/r2/" /> -->
+  <xacro:property name="robot_name" value= "/r2/"/>
   <include filename="$(find r2_description)/urdf/models/r2c_full_body_no_world.urdf.xacro" />
-  <xacro:robot_world_origin>
+  <!-- <xacro:robot_world_origin> -->
+  <xacro:macro name="robot_world_origin">
     <origin rpy="0 0 -1.57079" xyz="0.255 0.9 1.365"/>
 <!--    <origin rpy="0 0 0" xyz="0.5 0.7 1.212"/>-->
-  </xacro:robot_world_origin>
+  </xacro:macro>
+  <!-- </xacro:robot_world_origin> -->
   <include filename="$(find r2_description)/urdf/r2.gazebo.xacro" />
   <include filename="$(find r2_description)/urdf/sensors/r2.gazebo.sensors.xacro" />

File: r2_description/robots/r2c_full_body_no_world.urdf.xacro (robot description, xacro)
@@ -1,5 +1,6 @@
 <?xml version="1.0" ?>
-<robot name="r2c_full_body" xmlns:xacro="http://playerstage.sourceforge.net/gazebo/xmlschema/#interface">
-  <property name="robot_name" value= "/r2/" />
+<robot name="r2c_full_body" xmlns:xacro="http://www.ros.org/wiki/xacro">
+  <!-- <property name="robot_name" value= "/r2/" /> -->
+  <xacro:property name="robot_name" value= "/r2/"/>
   <non_visual_link name="${robot_name}robot_world"/>
   <xacro:macro name="robot_base_origin" params="*origin">

File: r2_description/robots/r2c_legs.display.urdf.xacro (robot description, xacro)
@@ -1,11 +1,12 @@
 <?xml version="1.0" ?>
-<robot name="r2c_legs" xmlns:controller="http://playerstage.sourceforge.net/gazebo/xmlschema/#controller"
-			xmlns:interface="http://playerstage.sourceforge.net/gazebo/xmlschema/#interface"
-			xmlns:sensor="http://playerstage.sourceforge.net/gazebo/xmlschema/#sensor"
-			xmlns:xacro="http://playerstage.sourceforge.net/gazebo/xmlschema/#interface">
-  <property name="robot_name" value= "/r2/" />
-  <include filename="$(find r2_description/urdf/models/r2c_legs.urdf.xacro" />
-  <include filename="$(find r2_description/urdf/r2c_legs.gazebo.xacro" />
-  <include filename="$(find r2_description/urdf/sensors/r2c_legs.gazebo.sensors.xacro" />
+<robot name="r2c_legs" xmlns:controller="http://www.ros.org/wiki/controller"
+			xmlns:interface="http://www.ros.org/wiki/interface"
+			xmlns:sensor="http://www.ros.org/wiki/sensor"
+			xmlns:xacro="http://www.ros.org/wiki/xacro">
+  <!-- <property name="robot_name" value= "/r2/" /> -->
+  <xacro:property name="robot_name" value= "/r2/"/>
+  <include filename="$(find r2_description)/urdf/models/r2c_legs.urdf.xacro" />
+  <include filename="$(find r2_description)/urdf/r2c_legs.gazebo.xacro" />
+  <include filename="$(find r2_description)/urdf/sensors/r2c_legs.gazebo.sensors.xacro" />
   <!--<include filename="$(find r2_description)/urdf/gazebo_plugins/gazebo_interface.xacro" />-->
   <include filename="$(find r2_description)/urdf/gazebo_plugins/leg_grippers.xacro" />

File: r2_description/robots/r2c_legs.sim.urdf.xacro (robot description, xacro)
@@ -1,8 +1,9 @@
 <?xml version="1.0" ?>
-<robot name="r2c_legs" xmlns:controller="http://playerstage.sourceforge.net/gazebo/xmlschema/#controller"
-			xmlns:interface="http://playerstage.sourceforge.net/gazebo/xmlschema/#interface"
-			xmlns:sensor="http://playerstage.sourceforge.net/gazebo/xmlschema/#sensor"
-			xmlns:xacro="http://playerstage.sourceforge.net/gazebo/xmlschema/#interface">
-  <property name="robot_name" value= "/r2/" />
+<robot name="r2c_legs" xmlns:controller="http://www.ros.org/wiki/controller"
+			xmlns:interface="http://www.ros.org/wiki/interface"
+			xmlns:sensor="http://www.ros.org/wiki/sensor"
+			xmlns:xacro="http://www.ros.org/wiki/xacro">
+  <!-- <property name="robot_name" value= "/r2/" /> -->
+  <xacro:property name="robot_name" value= "/r2/"/>
   <include filename="$(find r2_description)/urdf/models/r2c_legs.urdf.xacro" />
   <include filename="$(find r2_description)/urdf/r2c_legs.gazebo.xacro" />

File: r2_description/robots/r2c_legs.urdf.xacro (robot description, xacro)
@@ -1,5 +1,6 @@
 <?xml version="1.0" ?>
-<robot name="r2c_legs">
-  <property name="robot_name" value= "/r2/" />
+<robot name="r2c_legs" xmlns:xacro="http://www.ros.org/wiki/xacro">
+  <!-- <property name="robot_name" value= "/r2/" /> -->
+  <xacro:property name="robot_name" value= "/r2/"/>
   <include filename="$(find r2_description)/urdf/r2.common.xacro" />
   <include filename="$(find r2_description)/urdf/r2c_legs/r2c_legs.stand.xacro" />

File: r2_description/robots/r2c_legs_control.urdf.xacro (robot description, xacro)
@@ -1,5 +1,6 @@
 <?xml version="1.0" ?>
-<robot name="r2c_legs">
-  <property name="robot_name" value= "/r2/" />
+<robot name="r2c_legs" xmlns:xacro="http://www.ros.org/wiki/xacro">
+  <!-- <property name="robot_name" value= "/r2/" /> -->
+  <xacro:property name="robot_name" value= "/r2/"/>
   <link name="${robot_name}robot_world"/>
   <non_visual_link name="${robot_name}robot_base"/>

File: r2_description/robots/r2c_torso.sim.urdf.xacro (robot description, xacro)
@@ -1,8 +1,9 @@
 <?xml version="1.0" ?>
-<robot name="r2_torso" xmlns:controller="http://playerstage.sourceforge.net/gazebo/xmlschema/#controller"
-			xmlns:interface="http://playerstage.sourceforge.net/gazebo/xmlschema/#interface"
-			xmlns:sensor="http://playerstage.sourceforge.net/gazebo/xmlschema/#sensor"
-			xmlns:xacro="http://playerstage.sourceforge.net/gazebo/xmlschema/#interface">
-  <property name="robot_name" value= "/r2/" />
+<robot name="r2_torso" xmlns:controller="http://www.ros.org/wiki/controller"
+			xmlns:interface="http://www.ros.org/wiki/interface"
+			xmlns:sensor="http://www.ros.org/wiki/sensor"
+			xmlns:xacro="http://www.ros.org/wiki/xacro">
+  <!-- <property name="robot_name" value= "/r2/" /> -->
+  <xacro:property name="robot_name" value= "/r2/"/>
   <include filename="$(find r2_description)/urdf/models/r2c_upper_body_stand.urdf.xacro" />
   <include filename="$(find r2_description)/urdf/r2.gazebo.xacro" />
